File: ProTrinket doubleHPdisplay.sch (EAGLE design)
At the start: 14 parts

Commit message: routed board (thx jaromir)
Connections:
- net A0: now also U$1.CAT_4
- net A1: now also R4.2
- net A2: now also U$2.CAT_3
- net A3: now also R8.2
- net A4: now also R7.2
- net A5: now also U$2.CAT_4
- net D10: now also R1.2
- net D11: now also R5.2
- net D12: now also U$1.CAT_2
- net D13: now also U$1.CAT_3
- net D3: now also U$2.CAT_2
- net D4: now also R6.2
- net D5: now also U$2.CAT_1
- net D6: now also R3.2
- net D8: now also R2.2
- net D9: now also U$1.CAT_1
Changed lines of the file:
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@@
 <?xml version="1.0" encoding="utf-8"?>
 <!DOCTYPE eagle SYSTEM "eagle.dtd">
-<eagle version="6.5.0">
+<eagle version="6.4">
 <drawing>
 <settings>
@@
 <label x="139.7" y="190.5" size="1.778" layer="95"/>
 </segment>
+<segment>
+<pinref part="R1" gate="G$1" pin="2"/>
+<wire x1="119.38" y1="154.94" x2="121.92" y2="154.94" width="0.1524" layer="91"/>
+<label x="121.92" y="154.94" size="1.778" layer="95"/>
+</segment>
 </net>
 <net name="D11" class="0">
@@
 <label x="139.7" y="187.96" size="1.778" layer="95"/>
 </segment>
+<segment>
+<pinref part="R5" gate="G$1" pin="2"/>
+<wire x1="119.38" y1="144.78" x2="121.92" y2="144.78" width="0.1524" layer="91"/>
+<label x="121.92" y="144.78" size="1.778" layer="95"/>
+</segment>
 </net>
 <net name="D12" class="0">
@@
 <label x="139.7" y="185.42" size="1.778" layer="95"/>
 </segment>
+<segment>
+<pinref part="U$1" gate="G$1" pin="CAT_2"/>
+<wire x1="68.58" y1="152.4" x2="63.5" y2="152.4" width="0.1524" layer="91"/>
+<label x="58.42" y="152.4" size="1.778" layer="95"/>
+</segment>
 </net>
 <net name="D13" class="0">
@@
 <label x="139.7" y="182.88" size="1.778" layer="95"/>
 </segment>
+<segment>
+<pinref part="U$1" gate="G$1" pin="CAT_3"/>
+<wire x1="68.58" y1="149.86" x2="63.5" y2="149.86" width="0.1524" layer="91"/>
+<label x="58.42" y="149.86" size="1.778" layer="95"/>
+</segment>
 </net>
 <net name="A0" class="0">
@@
 <label x="139.7" y="177.8" size="1.778" layer="95"/>
 </segment>
+<segment>
+<pinref part="U$1" gate="G$1" pin="CAT_4"/>
+<wire x1="68.58" y1="147.32" x2="63.5" y2="147.32" width="0.1524" layer="91"/>
+<label x="58.42" y="147.32" size="1.778" layer="95"/>
+</segment>
 </net>
 <net name="A1" class="0">
@@
 <label x="139.7" y="175.26" size="1.778" layer="95"/>
 </segment>
+<segment>
+<pinref part="R4" gate="G$1" pin="2"/>
+<wire x1="119.38" y1="147.32" x2="121.92" y2="147.32" width="0.1524" layer="91"/>
+<label x="121.92" y="147.32" size="1.778" layer="95"/>
+</segment>
 </net>
 <net name="A2" class="0">
@@
 <label x="139.7" y="172.72" size="1.778" layer="95"/>
 </segment>
+<segment>
+<pinref part="U$2" gate="G$1" pin="CAT_3"/>
+<wire x1="68.58" y1="124.46" x2="63.5" y2="124.46" width="0.1524" layer="91"/>
+<label x="58.42" y="124.46" size="1.778" layer="95"/>
+</segment>
 </net>
 <net name="A3" class="0">
@@
 <label x="139.7" y="170.18" size="1.778" layer="95"/>
 </segment>
+<segment>
+<pinref part="R8" gate="G$1" pin="2"/>
+<wire x1="119.38" y1="137.16" x2="121.92" y2="137.16" width="0.1524" layer="91"/>
+<label x="121.92" y="137.16" size="1.778" layer="95"/>
+</segment>
 </net>
 <net name="A4" class="0">
@@
 <label x="139.7" y="167.64" size="1.778" layer="95"/>
 </segment>
+<segment>
+<pinref part="R7" gate="G$1" pin="2"/>
+<wire x1="119.38" y1="139.7" x2="121.92" y2="139.7" width="0.1524" layer="91"/>
+<label x="121.92" y="139.7" size="1.778" layer="95"/>
+</segment>
 </net>
 <net name="A5" class="0">
@@
 <label x="139.7" y="165.1" size="1.778" layer="95"/>
 </segment>
+<segment>
+<pinref part="U$2" gate="G$1" pin="CAT_4"/>
+<wire x1="68.58" y1="121.92" x2="63.5" y2="121.92" width="0.1524" layer="91"/>
+<label x="58.42" y="121.92" size="1.778" layer="95"/>
+</segment>
 </net>
 <net name="D3" class="0">
@@
 <pinref part="JP1" gate="G$1" pin="9"/>
 </segment>
+<segment>
+<pinref part="U$2" gate="G$1" pin="CAT_2"/>
+<wire x1="68.58" y1="127" x2="63.5" y2="127" width="0.1524" layer="91"/>
+<label x="58.42" y="127" size="1.778" layer="95"/>
+</segment>
 </net>
 <net name="D4" class="0">
@@
 <pinref part="JP1" gate="G$1" pin="8"/>
 </segment>
+<segment>
+<pinref part="R6" gate="G$1" pin="2"/>
+<wire x1="119.38" y1="142.24" x2="121.92" y2="142.24" width="0.1524" layer="91"/>
+<label x="121.92" y="142.24" size="1.778" layer="95"/>
+</segment>
 </net>
 <net name="D6" class="0">
@@
 <pinref part="JP1" gate="G$1" pin="6"/>
 </segment>
+<segment>
+<pinref part="R3" gate="G$1" pin="2"/>
+<wire x1="119.38" y1="149.86" x2="121.92" y2="149.86" width="0.1524" layer="91"/>
+<label x="121.92" y="149.86" size="1.778" layer="95"/>
+</segment>
 </net>
 <net name="D5" class="0">
@@
 <pinref part="JP1" gate="G$1" pin="7"/>
 </segment>
+<segment>
+<pinref part="U$2" gate="G$1" pin="CAT_1"/>
+<wire x1="68.58" y1="129.54" x2="63.5" y2="129.54" width="0.1524" layer="91"/>
+<label x="58.42" y="129.54" size="1.778" layer="95"/>
+</segment>
 </net>
 <net name="TXD" class="0">
@@
 <label x="162.56" y="182.88" size="1.778" layer="95"/>
 </segment>
+<segment>
+<pinref part="R2" gate="G$1" pin="2"/>
+<wire x1="119.38" y1="152.4" x2="121.92" y2="152.4" width="0.1524" layer="91"/>
+<label x="121.92" y="152.4" size="1.778" layer="95"/>
+</segment>
 </net>
 <net name="D9" class="0">
@@
 <label x="139.7" y="193.04" size="1.778" layer="95"/>
 </segment>
-</net>
+<segment>
+<pinref part="U$1" gate="G$1" pin="CAT_1"/>
+<wire x1="68.58" y1="154.94" x2="63.5" y2="154.94" width="0.1524" layer="91"/>
+<label x="58.42" y="154.94" size="1.778" layer="95"/>
+</segment>
+</net>
